File: centralHub_powerSupply/_autosave-centralHub_powerSupply.sch (KiCad schematic (older format))
At the start: 11 parts, among them J1 Screw_Terminal_01x02, J2 Screw_Terminal_01x02

Commit message: [Power Supply PCBS DONE!]
Parts:
- C1: footprint (none) -> Capacitor_THT:CP_Radial_D6.3mm_P2.50mm
- C2: footprint (none) -> Capacitor_THT:CP_Radial_D10.0mm_P5.00mm
- J1, J2: footprint (none) -> TerminalBlock:TerminalBlock_bornier-2_P5.08mm
- L1: footprint (none) -> Inductor_THT:L_Toroid_Vertical_L16.4mm_W7.6mm_P6.60mm_Vishay_TJ3
- U1: renamed from U?; footprint Package_TO_SOT_THT:TO-220-5_Vertical -> Package_TO_SOT_THT:TO-220-5_P3.4x3.7mm_StaggerOdd_Lead3.8mm_Vertical
Changed lines of the file:
@@
 F 0 "L1" V 7119 2300 50  0000 C CNN
 F 1 "100uH" V 7210 2300 50  0000 C CNN
-F 2 "" H 7300 2300 50  0001 C CNN
+F 2 "Inductor_THT:L_Toroid_Vertical_L16.4mm_W7.6mm_P6.60mm_Vishay_TJ3" H 7300 2300 50  0001 C CNN
 F 3 "~" H 7300 2300 50  0001 C CNN
 	1    7300 2300
@@
 F 0 "C1" H 5165 2446 50  0000 L CNN
 F 1 "100uF" H 5165 2355 50  0000 L CNN
-F 2 "" H 5050 2400 50  0001 C CNN
+F 2 "Capacitor_THT:CP_Radial_D6.3mm_P2.50mm" H 5050 2400 50  0001 C CNN
 F 3 "~" H 5050 2400 50  0001 C CNN
 	1    5050 2400
@@
 F 0 "C2" H 7765 2596 50  0000 L CNN
 F 1 "1000uF" H 7765 2505 50  0000 L CNN
-F 2 "" H 7650 2550 50  0001 C CNN
+F 2 "Capacitor_THT:CP_Radial_D10.0mm_P5.00mm" H 7650 2550 50  0001 C CNN
 F 3 "~" H 7650 2550 50  0001 C CNN
 	1    7650 2550
@@
 F 0 "J1" H 5180 3142 50  0000 L CNN
 F 1 "Screw_Terminal_01x02" H 5180 3051 50  0000 L CNN
-F 2 "" H 5100 3150 50  0001 C CNN
+F 2 "TerminalBlock:TerminalBlock_bornier-2_P5.08mm" H 5100 3150 50  0001 C CNN
 F 3 "~" H 5100 3150 50  0001 C CNN
 	1    5100 3150
@@
 F 0 "J2" H 7280 3192 50  0000 L CNN
 F 1 "Screw_Terminal_01x02" H 7280 3101 50  0000 L CNN
-F 2 "" H 7200 3200 50  0001 C CNN
+F 2 "TerminalBlock:TerminalBlock_bornier-2_P5.08mm" H 7200 3200 50  0001 C CNN
 F 3 "~" H 7200 3200 50  0001 C CNN
 	1    7200 3200
@@
 	6850 3300 7000 3300
 $Comp
-L Regulator_Switching:LM2576HVT-5 U?
+L Regulator_Switching:LM2576HVT-5 U1
 U 1 1 5DC1A549
 P 6200 2200
-F 0 "U?" H 6200 2567 50  0000 C CNN
+F 0 "U1" H 6200 2567 50  0000 C CNN
 F 1 "LM2576HVT-5" H 6200 2476 50  0000 C CNN
-F 2 "Package_TO_SOT_THT:TO-220-5_Vertical" H 6200 1950 50  0001 L CIN
+F 2 "Package_TO_SOT_THT:TO-220-5_P3.4x3.7mm_StaggerOdd_Lead3.8mm_Vertical" H 6200 1950 50  0001 L CIN
 F 3 "http://www.ti.com/lit/ds/symlink/lm2576.pdf" H 6200 2200 50  0001 C CNN
 	1    6200 2200
