File: centralHub_powerSupply/centralHub_powerSupply.kicad_pcb (KiCad board)
At the start: 2 copper layers, 100 x 50 mm, 11 parts, among them J1 Screw_Terminal_01x02, J2 Screw_Terminal_01x02, U1 LM2576HVT-5

Commit message: [PCB ESP32 e NRF]
Parts:
- moved C2 19.4 mm to (170.2, 92.7)
- moved L1 19.4 mm to (205.7, 87.6)
- moved D4 19.4 mm to (146.1, 72.4)
- moved J2 19.4 mm to (205.7, 71.1)
- moved J1 19.4 mm to (138.4, 101.6)
- moved D2 19.4 mm to (138.4, 72.4)
- moved D1 19.4 mm to (129.5, 87.6)
- moved D3 19.4 mm to (154.9, 87.6)
- moved C1 19.4 mm to (185.4, 90.2)
- moved D5 19.4 mm to (185.4, 72.4)
- moved U1 19.4 mm to (199.4, 97.8)
Routing:
- net +5V: track 101.2 -> 100.4 mm
- net (no net): vias 0 -> 4
