File: PCB_Medidores/PCB_Medidores.kicad_pcb (KiCad board)
At the start: 2 copper layers, 100 x 60 mm, 15 parts, among them J1 Screw_Terminal_01x02, SW1 SW_Push, U1 SENO, U2 tp4056, U3 DS18B20, U4 ATmega328P-PU, U5 NRF24L01_Breakout

Commit message: [PCB medidores V2.0]
-Correçao da PCB e melhorias
Parts:
- U4: footprint Package_DIP:DIP-28_W7.62mm -> Package_DIP:DIP-28_W7.62mm_LongPads
Routing:
- net +3V8: track 174.3 -> 195.1 mm
