File: PCB_Medidores/PCB_Medidores.sch (KiCad schematic (older format))
At the start: 20 parts, among them SW1 SW_Push, U1 SENO, U2 tp4056, U3 DS18B20, U4 ATmega8L-8PU, U5 EL814, U6 NRF24L01_Breakout, Y1 16MHz

Commit message: [PCB]
Parts:
- BT1: footprint (none) -> PI2_footprint:BatteryHolder
- C1: footprint (none) -> Capacitor_THT:CP_Radial_D6.3mm_P2.50mm
- C2, C3: footprint (none) -> Capacitor_THT:C_Disc_D3.0mm_W1.6mm_P2.50mm
- D2: footprint (none) -> Diode_THT:D_DO-41_SOD81_P10.16mm_Horizontal
- R1, R2, R3, R4, R5: footprint (none) -> Resistor_THT:R_Axial_DIN0204_L3.6mm_D1.6mm_P5.08mm_Horizontal
- SC1: footprint (none) -> Connector_JST:JST_XH_B2B-XH-A_1x02_P2.50mm_Vertical
- SW1: footprint (none) -> Button_Switch_THT:SW_PUSH_6mm_H4.3mm
- U1: footprint (none) -> Connector_JST:JST_XH_B3B-XH-A_1x03_P2.50mm_Vertical
- U2: footprint (none) -> PI2_footprint:tp4056
- U3: footprint Package_TO_SOT_THT:TO-92_Inline -> Connector_JST:JST_XH_B3B-XH-A_1x03_P2.50mm_Vertical
- U5: footprint (none) -> Package_DIP:DIP-4_W7.62mm
- Y1: footprint (none) -> Crystal:Crystal_HC52-6mm_Vertical
Changed lines of the file:
@@
 EESchema Schematic File Version 4
+LIBS:PCB_Medidores-cache
 EELAYER 30 0
 EELAYER END
@@
 F 0 "BT1" H 3618 2446 50  0000 L CNN
 F 1 "3.7V" H 3618 2355 50  0000 L CNN
-F 2 "" V 3500 2410 50  0001 C CNN
+F 2 "PI2_footprint:BatteryHolder" V 3500 2410 50  0001 C CNN
 F 3 "~" V 3500 2410 50  0001 C CNN
 	1    3500 2350
@@
 F 0 "SC1" H 2058 2446 50  0000 L CNN
 F 1 "Solar_Cell" H 2058 2355 50  0000 L CNN
-F 2 "" V 1950 2410 50  0001 C CNN
+F 2 "Connector_JST:JST_XH_B2B-XH-A_1x02_P2.50mm_Vertical" V 1950 2410 50  0001 C CNN
 F 3 "~" V 1950 2410 50  0001 C CNN
 	1    1950 2350
@@
 F 0 "Y1" V 5346 2519 50  0000 R CNN
 F 1 "16MHz" V 5255 2519 50  0000 R CNN
-F 2 "" H 5300 2650 50  0001 C CNN
+F 2 "Crystal:Crystal_HC52-6mm_Vertical" H 5300 2650 50  0001 C CNN
 F 3 "~" H 5300 2650 50  0001 C CNN
 	1    5300 2650
@@
 F 0 "R2" H 5509 2096 50  0000 L CNN
 F 1 "10k" H 5509 2005 50  0000 L CNN
-F 2 "" H 5450 2050 50  0001 C CNN
+F 2 "Resistor_THT:R_Axial_DIN0204_L3.6mm_D1.6mm_P5.08mm_Horizontal" H 5450 2050 50  0001 C CNN
 F 3 "~" H 5450 2050 50  0001 C CNN
 	1    5450 2050
@@
 F 0 "C1" H 3991 2346 50  0000 L CNN
 F 1 "100uF" H 3991 2255 50  0000 L CNN
-F 2 "" H 3900 2300 50  0001 C CNN
+F 2 "Capacitor_THT:CP_Radial_D6.3mm_P2.50mm" H 3900 2300 50  0001 C CNN
 F 3 "~" H 3900 2300 50  0001 C CNN
 	1    3900 2300
@@
 F 0 "U3" H 3320 4046 50  0000 R CNN
 F 1 "DS18B20" H 3320 3955 50  0000 R CNN
-F 2 "Package_TO_SOT_THT:TO-92_Inline" H 2550 3750 50  0001 C CNN
+F 2 "Connector_JST:JST_XH_B3B-XH-A_1x03_P2.50mm_Vertical" H 2550 3750 50  0001 C CNN
 F 3 "http://datasheets.maximintegrated.com/en/ds/DS18B20.pdf" H 3400 4250 50  0001 C CNN
 	1    3550 4000
@@
 F 0 "U2" H 2925 2225 50  0000 C CNN
 F 1 "tp4056" H 2925 2134 50  0000 C CNN
-F 2 "" H 2900 2100 50  0001 C CNN
+F 2 "PI2_footprint:tp4056" H 2900 2100 50  0001 C CNN
 F 3 "" H 2900 2100 50  0001 C CNN
 	1    2900 2100
@@
 F 0 "SW1" H 4950 2635 50  0000 C CNN
 F 1 "SW_Push" H 4950 2544 50  0000 C CNN
-F 2 "" H 4950 2550 50  0001 C CNN
+F 2 "Button_Switch_THT:SW_PUSH_6mm_H4.3mm" H 4950 2550 50  0001 C CNN
 F 3 "~" H 4950 2550 50  0001 C CNN
 	1    4950 2350
@@
 F 0 "C3" H 5392 3046 50  0000 L CNN
 F 1 "22pF" H 5392 2955 50  0000 L CNN
-F 2 "" H 5300 3000 50  0001 C CNN
+F 2 "Capacitor_THT:C_Disc_D3.0mm_W1.6mm_P2.50mm" H 5300 3000 50  0001 C CNN
 F 3 "~" H 5300 3000 50  0001 C CNN
 	1    5300 3000
@@
 F 0 "C2" H 4992 3046 50  0000 L CNN
 F 1 "22pF" H 4992 2955 50  0000 L CNN
-F 2 "" H 4900 3000 50  0001 C CNN
+F 2 "Capacitor_THT:C_Disc_D3.0mm_W1.6mm_P2.50mm" H 4900 3000 50  0001 C CNN
 F 3 "~" H 4900 3000 50  0001 C CNN
 	1    4900 3000
@@
 F 0 "U1" H 1956 3446 50  0000 R CNN
 F 1 "SENO" H 1956 3355 50  0000 R CNN
-F 2 "" H 2200 3700 50  0001 C CNN
+F 2 "Connector_JST:JST_XH_B3B-XH-A_1x03_P2.50mm_Vertical" H 2200 3700 50  0001 C CNN
 F 3 "" H 2200 3700 50  0001 C CNN
 	1    2200 3700
@@
 F 0 "R1" H 3159 3846 50  0000 L CNN
 F 1 "4.7k" H 3159 3755 50  0000 L CNN
-F 2 "" H 3100 3800 50  0001 C CNN
+F 2 "Resistor_THT:R_Axial_DIN0204_L3.6mm_D1.6mm_P5.08mm_Horizontal" H 3100 3800 50  0001 C CNN
 F 3 "~" H 3100 3800 50  0001 C CNN
 	1    3100 3800
@@
 F 0 "R3" H 9459 1646 50  0000 L CNN
 F 1 "Rzener" H 9459 1555 50  0000 L CNN
-F 2 "" H 9400 1600 50  0001 C CNN
+F 2 "Resistor_THT:R_Axial_DIN0204_L3.6mm_D1.6mm_P5.08mm_Horizontal" H 9400 1600 50  0001 C CNN
 F 3 "~" H 9400 1600 50  0001 C CNN
 	1    9400 1600
@@
 F 0 "D2" V 9904 1968 50  0000 L CNN
 F 1 " 1N4728" V 9995 1968 50  0000 L CNN
-F 2 "" V 9950 1900 50  0001 C CNN
+F 2 "Diode_THT:D_DO-41_SOD81_P10.16mm_Horizontal" V 9950 1900 50  0001 C CNN
 F 3 "~" V 9950 1900 50  0001 C CNN
 	1    9950 1900
@@
 F 0 "R4" H 9559 4346 50  0000 L CNN
 F 1 "10k" H 9559 4255 50  0000 L CNN
-F 2 "" H 9500 4300 50  0001 C CNN
+F 2 "Resistor_THT:R_Axial_DIN0204_L3.6mm_D1.6mm_P5.08mm_Horizontal" H 9500 4300 50  0001 C CNN
 F 3 "~" H 9500 4300 50  0001 C CNN
 	1    9500 4300
@@
 F 0 "R5" H 9559 4646 50  0000 L CNN
 F 1 "33k" H 9559 4555 50  0000 L CNN
-F 2 "" H 9500 4600 50  0001 C CNN
+F 2 "Resistor_THT:R_Axial_DIN0204_L3.6mm_D1.6mm_P5.08mm_Horizontal" H 9500 4600 50  0001 C CNN
 F 3 "~" H 9500 4600 50  0001 C CNN
 	1    9500 4600
@@
 F 0 "U5" H 9100 4375 50  0000 C CNN
 F 1 "EL814" H 9100 4284 50  0000 C CNN
-F 2 "" H 8900 3850 50  0001 L CIN
+F 2 "Package_DIP:DIP-4_W7.62mm" H 8900 3850 50  0001 L CIN
 F 3 "http://www.everlight.com/file/ProductFile/EL814.pdf" H 9125 4050 50  0001 L CNN
 	1    9100 4050

Commit message: [PCB Medidores e Correção]
Parts:
- removed C2, C3: 22pF, Capacitor_THT:C_Disc_D3.0mm_W1.6mm_P2.50mm, symbol Device:C_Small
- removed D1: 1N4007, Diode_THT:D_DO-41_SOD81_P10.16mm_Horizontal, symbol Diode:1N4007
- removed R4: 10k, Resistor_THT:R_Axial_DIN0204_L3.6mm_D1.6mm_P5.08mm_Horizontal, symbol Device:R_Small
- removed R5: 33k, Resistor_THT:R_Axial_DIN0204_L3.6mm_D1.6mm_P5.08mm_Horizontal, symbol Device:R_Small
- removed U4: ATmega8L-8PU, Package_DIP:DIP-28_W7.62mm, symbol MCU_Microchip_ATmega:ATmega8L-8PU
- removed U5: EL814, Package_DIP:DIP-4_W7.62mm, symbol Isolator:EL814
- removed Y1: 16MHz, Crystal:Crystal_HC52-6mm_Vertical, symbol Device:Crystal
- added J1: Screw_Terminal_01x02, TerminalBlock:TerminalBlock_bornier-2_P5.08mm, symbol Connector:Screw_Terminal_01x02
- added RV1: R_POT_TRIM, Potentiometer_THT:Potentiometer_Bourns_3296W_Vertical, symbol Device:R_POT_TRIM
- added U4: ATmega328P-PU, Package_DIP:DIP-28_W7.62mm, symbol MCU_Microchip_ATmega:ATmega328P-PU
- R1, R2: footprint Resistor_THT:R_Axial_DIN0204_L3.6mm_D1.6mm_P5.08mm_Horizontal -> Resistor_THT:R_Axial_DIN0207_L6.3mm_D2.5mm_P10.16mm_Horizontal
- R3: footprint Resistor_THT:R_Axial_DIN0204_L3.6mm_D1.6mm_P5.08mm_Horizontal -> Resistor_THT:R_Axial_DIN0207_L6.3mm_D2.5mm_P15.24mm_Horizontal
- U1: footprint Connector_JST:JST_XH_B3B-XH-A_1x03_P2.50mm_Vertical -> Connector_PinHeader_2.54mm:PinHeader_1x03_P2.54mm_Vertical
- renumbered D2 to D1, U6 to U5
Connections:
- net +3V8: now also J1.1 (Pin_1), RV1.1, U4.20 (AVCC), U4.7 (VCC); no longer BT1.1 (+)
- net A0: now also U4.27 (PC4)
- net A1: now also RV1.2, U4.24 (PC1)
- net AT02: now also U4.28 (PC5)
- net AT05: now also U4.4 (PD2)
- net AT06: now also U4.5 (PD3)
- net AT08: now also U4.14 (PB0)
- net AT09: now also U4.15 (PB1)
- net AT10: now also U4.16 (PB2)
- net AT11: now also U4.17 (PB3)
- net AT12: now also U4.18 (PB4)
- net AT13: now also U4.19 (PB5)
- net GND: now also SW1.2, J1.2 (Pin_2), RV1.3, U4.22 (GND), U4.8 (GND); no longer BT1.2 (-), SW1.1
- net at R2.2: now also SW1.1, U4.1 (~RESET~/PC6); no longer SW1.2
- net at SC1.1 (+): now also U2.1 (IN+)
- no-connect marks 9 -> 14
Other:
- moved on the sheet: BT1, C1, R2, SC1, SW1, U2
