File: PCB_controllerHub/PCB_controllerHub.sch (KiCad schematic (older format))
At the start: 16 parts, among them J1 Conn_01x04_Female, J2 Conn_01x04_Female, J3 Screw_Terminal_01x02, Q1 TIP42, T1 Transformer_1P_SS, U1 Module_Relay

Commit message: [Power Supply PCBS DONE!]
Parts:
- removed J1, J2: Conn_01x04_Female, symbol Connector:Conn_01x04_Female
- added J2: Screw_Terminal_01x02, TerminalBlock:TerminalBlock_bornier-2_P5.08mm, symbol Connector:Screw_Terminal_01x02
- C1: footprint (none) -> Capacitor_THT:CP_Radial_D10.0mm_P5.00mm
- C2: footprint (none) -> Capacitor_THT:CP_Radial_D6.3mm_P2.50mm
- C3: footprint (none) -> Capacitor_THT:C_Rect_L7.2mm_W2.5mm_P5.00mm_FKS2_FKP2_MKS2_MKP2
- J1: renamed from J3; footprint (none) -> TerminalBlock:TerminalBlock_bornier-2_P5.08mm
- R1: footprint (none) -> Resistor_THT:R_Axial_DIN0309_L9.0mm_D3.2mm_P12.70mm_Horizontal
- R2: footprint (none) -> Resistor_THT:R_Axial_DIN0207_L6.3mm_D2.5mm_P10.16mm_Horizontal
- T1: footprint (none) -> PI2_footprint:Trafo_1A_6V
- U1: footprint (none) -> PI2_footprint:Module_relay
- renumbered D2 to D1, D4 to D2, D1 to D3, D3 to D4
Connections:
- net +5V: now also D2.1 (K), D4.1 (K), J2.1 (Pin_1); no longer D1.2 (A), D3.2 (A), J1.1 (Pin_1), T1.5 (SB)
- net GND: now also J2.2 (Pin_2)
- net at C1.2, Q1.2 (C), R1.2: now also D1.2 (A), D3.2 (A); no longer D2.1 (K), D4.1 (K)
- net AC1: now reaches D3.1 (K), D4.2 (A)
- net AC1: now also J1.1 (Pin_1), T1.5 (SB)
Other:
- moved on the sheet: C1, D1, D2, D3, D4

Commit message: Fix minor error in ControllerHub Power Supply & Git files cleanup
Connections:
- net AC1: no longer T1.5 (SB)
- net AC2: no longer T1.3 (SA)
- net at C2.2, R1.1: now also D5.2 (A), Q1.1 (B)
- no-connect marks 7 -> 9
Other:
- moved on the sheet: J1, R1, T1
Changed lines of the file:
@@
 	-1   0    0    1
 $EndComp
-$Comp
-L Device:Transformer_1P_SS T1
-U 1 1 5DB43B8F
-P 2650 2650
-F 0 "T1" H 2650 3031 50  0000 C CNN
-F 1 "Transformer_1P_SS" H 2650 2940 50  0000 C CNN
-F 2 "PI2_footprint:Trafo_1A_6V" H 2650 2650 50  0001 C CNN
-F 3 "~" H 2650 2650 50  0001 C CNN
-	1    2650 2650
-	1    0    0    -1
-$EndComp
 Wire Wire Line
 	4550 1550 4550 1700
 Wire Wire Line
 	4550 1700 4500 1700
-NoConn ~ 3050 2650
+NoConn ~ 5200 2600
 Wire Wire Line
 	4150 1700 4200 1700
@@
 	4150 1150 4200 1150
 Connection ~ 4150 1150
-NoConn ~ 2250 2450
-NoConn ~ 2250 2850
-Wire Wire Line
-	3050 2450 3150 2450
-Wire Wire Line
-	3150 2450 3150 2600
-Wire Wire Line
-	3150 2600 3200 2600
-Wire Wire Line
-	3050 2850 3150 2850
-Wire Wire Line
-	3150 2850 3150 2700
-Text GLabel 3500 2850 2    50   Input ~ 0
+NoConn ~ 4400 2400
+NoConn ~ 4400 2800
+Text GLabel 5650 2800 2    50   Input ~ 0
 AC2
 Wire Wire Line
-	3200 2600 3200 2450
-Wire Wire Line
-	3200 2450 3500 2450
-Connection ~ 3200 2600
-Wire Wire Line
-	3150 2700 3200 2700
-Wire Wire Line
-	3500 2850 3200 2850
-Wire Wire Line
-	3200 2850 3200 2700
-Connection ~ 3200 2700
+	5350 2400 5650 2400
+Wire Wire Line
+	5650 2800 5350 2800
+Wire Wire Line
+	5350 2800 5350 2650
 Text GLabel 3800 1800 0    50   Input ~ 0
 AC1
@@
 L Device:R_Small R1
 U 1 1 5DB96D2D
-P 5600 1550
-F 0 "R1" H 5659 1596 50  0000 L CNN
-F 1 "270" H 5659 1505 50  0000 L CNN
-F 2 "Resistor_THT:R_Axial_DIN0309_L9.0mm_D3.2mm_P12.70mm_Horizontal" H 5600 1550 50  0001 C CNN
-F 3 "~" H 5600 1550 50  0001 C CNN
-	1    5600 1550
+P 5600 1700
+F 0 "R1" H 5659 1746 50  0000 L CNN
+F 1 "270" H 5659 1655 50  0000 L CNN
+F 2 "Resistor_THT:R_Axial_DIN0309_L9.0mm_D3.2mm_P12.70mm_Horizontal" H 5600 1700 50  0001 C CNN
+F 3 "~" H 5600 1700 50  0001 C CNN
+	1    5600 1700
 	1    0    0    -1
 $EndComp
@@
 $EndComp
 Wire Wire Line
-	5600 1400 5600 1450
-Wire Wire Line
 	5600 1150 5600 1200
 Wire Wire Line
@@
 $EndComp
 Wire Wire Line
-	5800 1850 5600 1850
-Wire Wire Line
-	6000 1550 6000 1450
+	6000 1550 6000 1500
 $Comp
 L Device:R_Small R2
@@
 Connection ~ 6900 1850
 $Comp
+L Connector:Screw_Terminal_01x02 J1
+U 1 1 5DBF98DD
+P 5700 2550
+F 0 "J1" H 5780 2542 50  0000 L CNN
+F 1 "Screw_Terminal_01x02" H 5780 2451 50  0000 L CNN
+F 2 "TerminalBlock:TerminalBlock_bornier-2_P5.08mm" H 5700 2550 50  0001 C CNN
+F 3 "~" H 5700 2550 50  0001 C CNN
+	1    5700 2550
+	1    0    0    -1
+$EndComp
+Wire Wire Line
+	5350 2650 5500 2650
+Text GLabel 5650 2400 2    50   Input ~ 0
+AC1
+NoConn ~ 7050 2600
+NoConn ~ 7050 2700
+NoConn ~ 7050 2800
+$Comp
+L Connector:Screw_Terminal_01x02 J2
+U 1 1 5DBB1AFE
+P 7750 1450
+F 0 "J2" H 7830 1442 50  0000 L CNN
+F 1 "Screw_Terminal_01x02" H 7830 1351 50  0000 L CNN
+F 2 "TerminalBlock:TerminalBlock_bornier-2_P5.08mm" H 7750 1450 50  0001 C CNN
+F 3 "~" H 7750 1450 50  0001 C CNN
+	1    7750 1450
+	1    0    0    -1
+$EndComp
+Wire Wire Line
+	7550 1450 7350 1450
+Wire Wire Line
+	7350 1450 7350 1150
+Wire Wire Line
+	6900 1150 7350 1150
+Wire Wire Line
+	7350 1150 7550 1150
+Connection ~ 7350 1150
+Wire Wire Line
+	6900 1850 7350 1850
+Wire Wire Line
+	7550 1550 7350 1550
+Wire Wire Line
+	7350 1550 7350 1850
+Connection ~ 7350 1850
+Wire Wire Line
+	7350 1850 7550 1850
+Connection ~ 4550 1700
+Connection ~ 4550 1150
+Wire Wire Line
+	4550 1700 4550 1800
+Wire Wire Line
+	3800 1150 4150 1150
+Wire Wire Line
+	3800 1800 4550 1800
+Wire Wire Line
+	4150 1700 4150 1850
+Connection ~ 4150 1700
+Wire Wire Line
+	4550 1150 5050 1150
+Wire Wire Line
+	4150 1850 5050 1850
+Wire Wire Line
+	5050 1450 5050 1150
+Connection ~ 5050 1150
+Wire Wire Line
+	5050 1150 5600 1150
+Wire Wire Line
+	5050 1650 5050 1850
+Connection ~ 5050 1850
+NoConn ~ 7050 2500
+$Comp
 L PI2_Library:Module_Relay U1
 U 1 1 5DBC8D34
@@
 	1    0    0    -1
 $EndComp
-$Comp
-L Connector:Screw_Terminal_01x02 J1
-U 1 1 5DBF98DD
-P 3550 2600
-F 0 "J1" H 3630 2592 50  0000 L CNN
-F 1 "Screw_Terminal_01x02" H 3630 2501 50  0000 L CNN
-F 2 "TerminalBlock:TerminalBlock_bornier-2_P5.08mm" H 3550 2600 50  0001 C CNN
-F 3 "~" H 3550 2600 50  0001 C CNN
-	1    3550 2600
-	1    0    0    -1
-$EndComp
-Wire Wire Line
-	3200 2600 3350 2600
-Wire Wire Line
-	3200 2700 3350 2700
-Text GLabel 3500 2450 2    50   Input ~ 0
-AC1
-NoConn ~ 7050 2500
-NoConn ~ 7050 2600
-NoConn ~ 7050 2700
-NoConn ~ 7050 2800
-$Comp
-L Connector:Screw_Terminal_01x02 J2
-U 1 1 5DBB1AFE
-P 7750 1450
-F 0 "J2" H 7830 1442 50  0000 L CNN
-F 1 "Screw_Terminal_01x02" H 7830 1351 50  0000 L CNN
-F 2 "TerminalBlock:TerminalBlock_bornier-2_P5.08mm" H 7750 1450 50  0001 C CNN
-F 3 "~" H 7750 1450 50  0001 C CNN
-	1    7750 1450
-	1    0    0    -1
-$EndComp
-Wire Wire Line
-	7550 1450 7350 1450
-Wire Wire Line
-	7350 1450 7350 1150
-Wire Wire Line
-	6900 1150 7350 1150
-Wire Wire Line
-	7350 1150 7550 1150
-Connection ~ 7350 1150
-Wire Wire Line
-	6900 1850 7350 1850
-Wire Wire Line
-	7550 1550 7350 1550
-Wire Wire Line
-	7350 1550 7350 1850
-Connection ~ 7350 1850
-Wire Wire Line
-	7350 1850 7550 1850
-Connection ~ 4550 1700
-Connection ~ 4550 1150
-Wire Wire Line
-	4550 1700 4550 1800
-Wire Wire Line
-	5600 1650 5600 1850
+Wire Wire Line
+	5050 1850 5600 1850
+Wire Wire Line
+	5600 1400 5600 1500
+Wire Wire Line
+	5600 1800 5600 1850
 Connection ~ 5600 1850
 Wire Wire Line
-	3800 1150 4150 1150
-Wire Wire Line
-	3800 1800 4550 1800
-Wire Wire Line
-	4150 1700 4150 1850
-Connection ~ 4150 1700
-Wire Wire Line
-	4550 1150 5050 1150
-Wire Wire Line
-	4150 1850 5050 1850
-Wire Wire Line
-	5050 1450 5050 1150
-Connection ~ 5050 1150
-Wire Wire Line
-	5050 1150 5600 1150
-Wire Wire Line
-	5050 1650 5050 1850
-Connection ~ 5050 1850
-Wire Wire Line
-	5050 1850 5600 1850
+	5600 1850 5800 1850
+Wire Wire Line
+	5600 1500 6000 1500
+Connection ~ 5600 1500
+Wire Wire Line
+	5600 1500 5600 1600
+Connection ~ 6000 1500
+Wire Wire Line
+	6000 1500 6000 1450
+$Comp
+L Device:Transformer_1P_SS T1
+U 1 1 5DB43B8F
+P 4800 2600
+F 0 "T1" H 4800 2981 50  0000 C CNN
+F 1 "Transformer_1P_SS" H 4800 2890 50  0000 C CNN
+F 2 "PI2_footprint:Trafo_1A_6V" H 4800 2600 50  0001 C CNN
+F 3 "~" H 4800 2600 50  0001 C CNN
+	1    4800 2600
+	1    0    0    -1
+$EndComp
+Wire Wire Line
+	5350 2550 5500 2550
+Wire Wire Line
+	5350 2550 5350 2400
+NoConn ~ 5200 2800
+NoConn ~ 5200 2400
 $EndSCHEMATC
