File: pcbMedidores_V2.0/pcbMedidores_V2.0.kicad_pcb (KiCad board)
At the start: 2 copper layers, 104.1 x 61.3 mm, 22 parts, among them J1 Li-Ion Battery, J2 Conn_01x04_Female, SW1 SW_Push, U1 ATmega328P-PU, U2 Tp4056+, U3 DS18B20, U4 NRF24L01+, U5 SENO

Commit message: [Minor correction]
Parts:
- R3: footprint Resistor_THT:R_Axial_DIN0207_L6.3mm_D2.5mm_P15.24mm_Horizontal -> Resistor_THT:R_Axial_DIN0207_L6.3mm_D2.5mm_P7.62mm_Horizontal
Connections:
- U1 pad 27: Net-(U1-Pad27) -> GNDPWR
Changed lines of the file:
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@@
     (zones 0)
     (modules 22)
-    (nets 33)
+    (nets 32)
   )
   (page A)
@@
   )
   (setup
-    (last_trace_width 1)
+    (last_trace_width 0.25)
     (user_trace_width 1)
     (trace_clearance 0.2)
@@
     (mod_text_size 1 1)
     (mod_text_width 0.15)
-    (pad_size 7 7)
-    (pad_drill 3.5)
+    (pad_size 2.4 1.6)
+    (pad_drill 0.8)
     (pad_to_mask_clearance 0.051)
     (solder_mask_min_width 0.25)
@@
   (net 30 "Net-(U1-Pad25)")
   (net 31 "Net-(U1-Pad12)")
-  (net 32 "Net-(U1-Pad27)")
   (net_class Default "Esta é a classe de rede padrão."
     (clearance 0.2)
@@
     (add_net "Net-(U1-Pad23)")
     (add_net "Net-(U1-Pad25)")
-    (add_net "Net-(U1-Pad27)")
     (add_net "Net-(U1-Pad4)")
     (add_net "Net-(U1-Pad5)")
@@
     (add_net "Net-(U1-Pad9)")
     (add_net VBUS)
+  )
+  (module Resistor_THT:R_Axial_DIN0207_L6.3mm_D2.5mm_P7.62mm_Horizontal (layer F.Cu)
+    (at 160.02 72.39)
+    (descr "Resistor, Axial_DIN0207 series, Axial, Horizontal, pin pitch=7.62mm, 0.25W = 1/4W, length*diameter=6.3*2.5mm^2, http://cdn-reichelt.de/documents/datenblatt/B400/1_4W%23YAG.pdf")
+    (tags "Resistor Axial_DIN0207 series Axial Horizontal pin pitch 7.62mm 0.25W = 1/4W length 6.3mm diameter 2.5mm")
+    (fp_text reference R3 (at 7.62 -2.37) (layer F.SilkS)
+      (effects (font (size 1 1) (thickness 0.15)))
+    )
+    (fp_text value 100 (at 7.62 2.37) (layer F.Fab)
+      (effects (font (size 1 1) (thickness 0.15)))
+    )
+    (fp_text user %R (at 7.62 0) (layer F.Fab)
+      (effects (font (size 1 1) (thickness 0.15)))
+    )
+    (fp_line (start 8.67 -1.5) (end -1.05 -1.5) (layer F.CrtYd) (width 0.05))
+    (fp_line (start 8.67 1.5) (end 8.67 -1.5) (layer F.CrtYd) (width 0.05))
+    (fp_line (start -1.05 1.5) (end 8.67 1.5) (layer F.CrtYd) (width 0.05))
+    (fp_line (start -1.05 -1.5) (end -1.05 1.5) (layer F.CrtYd) (width 0.05))
+    (fp_line (start 7.08 1.37) (end 7.08 1.04) (layer F.SilkS) (width 0.12))
+    (fp_line (start 0.54 1.37) (end 7.08 1.37) (layer F.SilkS) (width 0.12))
+    (fp_line (start 0.54 1.04) (end 0.54 1.37) (layer F.SilkS) (width 0.12))
+    (fp_line (start 7.08 -1.37) (end 7.08 -1.04) (layer F.SilkS) (width 0.12))
+    (fp_line (start 0.54 -1.37) (end 7.08 -1.37) (layer F.SilkS) (width 0.12))
+    (fp_line (start 0.54 -1.04) (end 0.54 -1.37) (layer F.SilkS) (width 0.12))
+    (fp_line (start 7.62 0) (end 6.96 0) (layer F.Fab) (width 0.1))
+    (fp_line (start 0 0) (end 0.66 0) (layer F.Fab) (width 0.1))
+    (fp_line (start 6.96 -1.25) (end 0.66 -1.25) (layer F.Fab) (width 0.1))
+    (fp_line (start 6.96 1.25) (end 6.96 -1.25) (layer F.Fab) (width 0.1))
+    (fp_line (start 0.66 1.25) (end 6.96 1.25) (layer F.Fab) (width 0.1))
+    (fp_line (start 0.66 -1.25) (end 0.66 1.25) (layer F.Fab) (width 0.1))
+    (pad 2 thru_hole oval (at 7.62 0) (size 1.6 1.6) (drill 0.8) (layers *.Cu *.Mask)
+      (net 3 "Net-(D1-Pad1)"))
+    (pad 1 thru_hole circle (at 0 0) (size 1.6 1.6) (drill 0.8) (layers *.Cu *.Mask)
+      (net 1 VBUS))
+    (model ${KISYS3DMOD}/Resistor_THT.3dshapes/R_Axial_DIN0207_L6.3mm_D2.5mm_P7.62mm_Horizontal.wrl
+      (at (xyz 0 0 0))
+      (scale (xyz 1 1 1))
+      (rotate (xyz 0 0 0))
+    )
   )
   (module PI2_footprint:BatteryHolder (layer F.Cu)
@@
     (fp_line (start -39.03 15.91) (end 39.03 15.91) (layer F.CrtYd) (width 0.05))
     (fp_line (start 38.64 -5.36) (end -38.64 -5.36) (layer F.SilkS) (width 0.12))
-  )
-  (module Resistor_THT:R_Axial_DIN0207_L6.3mm_D2.5mm_P15.24mm_Horizontal (layer F.Cu)
-    (at 160.02 72.39)
-    (descr "Resistor, Axial_DIN0207 series, Axial, Horizontal, pin pitch=15.24mm, 0.25W = 1/4W, length*diameter=6.3*2.5mm^2, http://cdn-reichelt.de/documents/datenblatt/B400/1_4W%23YAG.pdf")
-    (tags "Resistor Axial_DIN0207 series Axial Horizontal pin pitch 15.24mm 0.25W = 1/4W length 6.3mm diameter 2.5mm")
-    (fp_text reference R3 (at 7.62 -2.37) (layer F.SilkS)
-      (effects (font (size 1 1) (thickness 0.15)))
-    )
-    (fp_text value 100 (at 7.62 2.37) (layer F.Fab)
-      (effects (font (size 1 1) (thickness 0.15)))
-    )
-    (fp_text user %R (at 7.62 0) (layer F.Fab)
-      (effects (font (size 1 1) (thickness 0.15)))
-    )
-    (fp_line (start 16.29 -1.5) (end -1.05 -1.5) (layer F.CrtYd) (width 0.05))
-    (fp_line (start 16.29 1.5) (end 16.29 -1.5) (layer F.CrtYd) (width 0.05))
-    (fp_line (start -1.05 1.5) (end 16.29 1.5) (layer F.CrtYd) (width 0.05))
-    (fp_line (start -1.05 -1.5) (end -1.05 1.5) (layer F.CrtYd) (width 0.05))
-    (fp_line (start 14.2 0) (end 10.89 0) (layer F.SilkS) (width 0.12))
-    (fp_line (start 1.04 0) (end 4.35 0) (layer F.SilkS) (width 0.12))
-    (fp_line (start 10.89 -1.37) (end 4.35 -1.37) (layer F.SilkS) (width 0.12))
-    (fp_line (start 10.89 1.37) (end 10.89 -1.37) (layer F.SilkS) (width 0.12))
-    (fp_line (start 4.35 1.37) (end 10.89 1.37) (layer F.SilkS) (width 0.12))
-    (fp_line (start 4.35 -1.37) (end 4.35 1.37) (layer F.SilkS) (width 0.12))
-    (fp_line (start 15.24 0) (end 10.77 0) (layer F.Fab) (width 0.1))
-    (fp_line (start 0 0) (end 4.47 0) (layer F.Fab) (width 0.1))
-    (fp_line (start 10.77 -1.25) (end 4.47 -1.25) (layer F.Fab) (width 0.1))
-    (fp_line (start 10.77 1.25) (end 10.77 -1.25) (layer F.Fab) (width 0.1))
-    (fp_line (start 4.47 1.25) (end 10.77 1.25) (layer F.Fab) (width 0.1))
-    (fp_line (start 4.47 -1.25) (end 4.47 1.25) (layer F.Fab) (width 0.1))
-    (pad 2 thru_hole oval (at 15.24 0) (size 1.6 1.6) (drill 0.8) (layers *.Cu *.Mask)
-      (net 3 "Net-(D1-Pad1)"))
-    (pad 1 thru_hole circle (at 0 0) (size 1.6 1.6) (drill 0.8) (layers *.Cu *.Mask)
-      (net 1 VBUS))
-    (model ${KISYS3DMOD}/Resistor_THT.3dshapes/R_Axial_DIN0207_L6.3mm_D2.5mm_P15.24mm_Horizontal.wrl
-      (at (xyz 0 0 0))
-      (scale (xyz 1 1 1))
-      (rotate (xyz 0 0 0))
-    )
   )
   (module PI2_footprint:Tp4056+ (layer B.Cu)
@@
       (net 4 /LED))
     (pad 27 thru_hole rect (at 7.62 2.54 90) (size 2.4 1.6) (drill 0.8) (layers *.Cu *.Mask)
-      (net 32 "Net-(U1-Pad27)"))
+      (net 2 GNDPWR))
     (pad 14 thru_hole oval (at 0 33.02 90) (size 2.4 1.6) (drill 0.8) (layers *.Cu *.Mask)
       (net 20 /CE))
@@
   (segment (start 153.67 107.95) (end 153.67 110.15) (width 1) (layer B.Cu) (net 1))
   (segment (start 149.86 66.04) (end 152.4 66.04) (width 1) (layer B.Cu) (net 1))
+  (segment (start 160.02 72.39) (end 158.75 72.39) (width 1) (layer B.Cu) (net 1))
   (segment (start 158.75 72.39) (end 152.4 66.04) (width 1) (layer B.Cu) (net 1))
-  (segment (start 160.02 72.39) (end 158.75 72.39) (width 1) (layer B.Cu) (net 1))
+  (segment (start 167.64 76.2) (end 181.61 76.2) (width 1) (layer B.Cu) (net 3))
   (segment (start 167.64 76.2) (end 167.64 72.39) (width 1) (layer B.Cu) (net 3))
-  (segment (start 167.64 76.2) (end 181.61 76.2) (width 1) (layer B.Cu) (net 3))
   (segment (start 163.83 119.38) (end 163.83 115.57) (width 1) (layer B.Cu) (net 4))
   (segment (start 107.99 71.12) (end 105.41 73.7) (width 1) (layer B.Cu) (net 5))
