File: pcbMedidores_V2.0/pcbMedidores_V2.0.sch (KiCad schematic (older format))
At the start: 18 parts, among them J1 Li-Ion Battery, J2 Conn_01x04_Female, SW1 SW_Push, U1 ATmega328P-PU, U2 Tp4056+, U3 DS18B20, U4 NRF24L01+, U5 SENO

Commit message: [Minor correction]
Parts:
- R3: footprint Resistor_THT:R_Axial_DIN0207_L6.3mm_D2.5mm_P15.24mm_Horizontal -> Resistor_THT:R_Axial_DIN0207_L6.3mm_D2.5mm_P7.62mm_Horizontal
Connections:
- net GNDPWR: now also U1.27 (PC4)
- no-connect marks 13 -> 12
Changed lines of the file:
@@
 F 0 "R3" H 7759 2996 50  0000 L CNN
 F 1 "100" H 7759 2905 50  0000 L CNN
-F 2 "Resistor_THT:R_Axial_DIN0207_L6.3mm_D2.5mm_P15.24mm_Horizontal" H 7700 2950 50  0001 C CNN
+F 2 "Resistor_THT:R_Axial_DIN0207_L6.3mm_D2.5mm_P7.62mm_Horizontal" H 7700 2950 50  0001 C CNN
 F 3 "~" H 7700 2950 50  0001 C CNN
 	1    7700 2950
@@
 NoConn ~ 3000 2350
 Wire Wire Line
-	2850 2550 3000 2550
-NoConn ~ 3000 2550
-Wire Wire Line
 	2850 3350 3000 3350
 NoConn ~ 3000 3350
@@
 Wire Wire Line
 	8900 5850 9150 5850
+$Comp
+L PI2_Library:GND #PWR?
+U 1 1 5E133A14
+P 3450 2550
+F 0 "#PWR?" H 3450 2350 50  0001 C CNN
+F 1 "GND" H 3459 2426 50  0000 C CNN
+F 2 "" H 3450 2500 50  0001 C CNN
+F 3 "" H 3450 2500 50  0001 C CNN
+	1    3450 2550
+	1    0    0    -1
+$EndComp
+Wire Wire Line
+	2850 2550 3450 2550
 $EndSCHEMATC
